File: hardware/electronics/PicoSynth.kicad_sch (KiCad schematic)
At the start: 160 parts, among them J1 Conn_01x06_Socket, J2 Micro_SD_Card, J3 Conn_01x04_Socket, J4 Conn_01x09_Socket, SW1 RotaryEncoder_Switch_MP, SW10 SW_Push_45deg, SW11 SW_Push_45deg, SW12 SW_Push_45deg, SW13 SW_Push_45deg, SW14 SW_Push_45deg, SW15 SW_Push_45deg, SW16 SW_Push_45deg, SW17 SW_Push_45deg, SW18 SW_Push_45deg, SW19 SW_Push_45deg, SW2 RotaryEncoder_Switch_MP, SW20 SW_Push_45deg, SW3 RotaryEncoder_Switch_MP, SW4 RotaryEncoder_Switch_MP, SW5 SW_Push_45deg, SW6 SW_Push_45deg, SW7 SW_Push_45deg, SW8 SW_Push_45deg, SW9 SW_Push_45deg, U1 Pico, U2 PCM5102A, U3 TC1262-33, U4 TC1262-33, U5 PCF8574, U6 PCF8574, U7 PCF8574, U8 AMS1117-3.3

Commit message: Basic routing almost complete: 6 more traces to go
Parts:
- removed R41: 10k, Cern_Ignition:R_0805_2012Metric_Pad1.20x1.40mm_HandSolder_modif, symbol Device:R_US
- added H1, H2, H3, H4: MountingHole_Pad, MountingHole:MountingHole_2.2mm_M2_Pad_Via, symbol Mechanical:MountingHole_Pad
- added J5: Line_Out, Connector_PinHeader_2.54mm:PinHeader_1x04_P2.54mm_Vertical, symbol Connector:Conn_01x04_Socket
- added J6: Conn_01x06_Socket, Connector_PinSocket_2.54mm:PinSocket_1x06_P2.54mm_Vertical, symbol Connector:Conn_01x06_Socket
- added R45, R46, R47, R48, R49, R50, R51, R52, R53, R54: 10k, Cern_Ignition:R_0805_2012Metric_Pad1.20x1.40mm_HandSolder_modif, symbol Device:R_US
- C33, C34, J2, R42, R43, R44: now not fitted; now left out of the parts list
- R31, R32: value 4.7k -> 10k
- U1: footprint Pi_Pico:RPi_Pico_SMD_TH -> Pi_Pico:RPi_Pico_SMD_TH_No_Debug
Connections:
- net +3V3: now also J6.1 (Pin_1); no longer R31.1, R32.1
- net +3V3_Pico: now also R31.2, R32.2, R45.2, R46.2, R47.2, R48.2, R49.2, R50.2, R51.2, R52.2, R53.2, R54.2
- net BCK: now also U1.16 (GPIO12); no longer U1.21 (GPIO16)
- net CLK: now also J6.4 (Pin_4)
- net DIN: now also U1.19 (GPIO14); no longer U1.24 (GPIO18)
- net Encoder0_A: now also R47.1
- net Encoder0_B: now also R48.1
- net Encoder0_Sw: now also R31.1
- net Encoder1_A: now also R51.1
- net Encoder1_B: now also R52.1
- net Encoder1_Sw: now also R46.1
- net Encoder2_A: now also R49.1
- net Encoder2_B: now also R50.1
- net Encoder2_Sw: now also R32.1
- net Encoder3_A: now also R54.1
- net Encoder3_B: now also R53.1
- net Encoder3_Sw: now also R45.1
- net GND: now also J2.9 (SHIELD), H1.1, H2.1, H3.1, H4.1, J6.6 (Pin_6)
- net L: now also J5.1 (Pin_1)
- net LRCK: now also U1.17 (GPIO13); no longer U1.22 (GPIO17)
- net Pin0: now also D2.1 (K), D3.1 (K), D4.1 (K), D5.1 (K); no longer SW13.1, SW14.1, SW5.1, SW9.1
- net Pin1: now also D6.1 (K), D7.1 (K), D8.1 (K), D9.1 (K); no longer SW10.1, SW15.1, SW16.1, SW6.1
- net Pin2: now also SW13.1, SW14.1, SW5.1, SW9.1; no longer SW11.1, SW17.1, SW18.1, SW7.1
- net Pin3: now also SW10.1, SW15.1, SW16.1, SW6.1; no longer SW12.1, SW19.1, SW20.1, SW8.1
- net Pin4: now also D11.1 (K), D13.1 (K), D15.1 (K), D17.1 (K); no longer D2.1 (K), D3.1 (K), D4.1 (K), D5.1 (K)
- net Pin5: now also SW11.1, SW17.1, SW18.1, SW7.1; no longer D6.1 (K), D7.1 (K), D8.1 (K), D9.1 (K)
- net Pin7: now also SW12.1, SW19.1, SW20.1, SW8.1; no longer D11.1 (K), D13.1 (K), D15.1 (K), D17.1 (K)
- net R: now also J5.3 (Pin_3)
- net SCL_Bus_0: now also R7.2, U1.22 (GPIO17), U5.14 (SCL); no longer J3.3 (Pin_3), R22.2, R32.2, U6.14 (SCL), U7.14 (SCL)
- net SCL_Bus_1: now also J3.3 (Pin_3), R22.2, U1.32 (GPIO27_ADC1), U6.14 (SCL), U7.14 (SCL); no longer R7.2, U5.14 (SCL)
- net SDA_Bus_0: now also R8.2, U1.21 (GPIO16), U5.15 (SDA); no longer J3.4 (Pin_4), R21.2, R31.2, U6.15 (SDA), U7.15 (SDA)
- net SDA_Bus_1: now also J3.4 (Pin_4), R21.2, U1.31 (GPIO26_ADC0), U6.15 (SDA), U7.15 (SDA); no longer R8.2, U5.15 (SDA)
- net G renamed G_L
- net G_L: now also J5.2 (Pin_2); no longer J4.4 (Pin_4)
- new net CS: J6.2 (Pin_2)
- new net G_R: J4.4 (Pin_4), J5.4 (Pin_4)
- new net MISO: J6.5 (Pin_5)
- new net MOSI: J6.3 (Pin_3)
- no-connect marks 8 -> 9
Other:
- note added: "Cheaper to buy the SD card module..."
- note added: "No pull-up resistor here Not needed because they are connected to the same bus as the other LEDs"
- note removed: "Do not forget to set the pull-up resistors in the GPIO"
- moved on the sheet: C15, C16, C17, C18, C19, C20, C21, C22, C23, C24, C25, C26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

Commit message: Routing Done, to-do: verify schematic and fix silkscreen
Parts:
- added J10, J11, J12, J13, J14, J9: Conn_01x14_Socket, Connector_PinHeader_2.54mm:PinHeader_1x14_P2.54mm_Vertical, symbol Connector:Conn_01x14_Socket
- added J7, J8: Conn_01x01_Socket, Connector_PinHeader_2.54mm:PinHeader_1x01_P2.54mm_Vertical, symbol Connector:Conn_01x01_Socket
Connections:
- net +3V3: now also J9.1 (Pin_1), J9.10 (Pin_10), J9.11 (Pin_11), J9.12 (Pin_12), J9.13 (Pin_13), J9.14 (Pin_14), J9.2 (Pin_2), J9.3 (Pin_3), J9.4 (Pin_4), J9.5 (Pin_5), J9.6 (Pin_6), J9.7 (Pin_7), J9.8 (Pin_8), J9.9 (Pin_9)
- net CLK: now also U1.24 (GPIO18)
- net CS: now also U1.22 (GPIO17)
- net GND: now also J10.1 (Pin_1), J10.10 (Pin_10), J10.11 (Pin_11), J10.12 (Pin_12), J10.13 (Pin_13), J10.14 (Pin_14), J10.2 (Pin_2), J10.3 (Pin_3), J10.4 (Pin_4), J10.5 (Pin_5), J10.6 (Pin_6), J10.7 (Pin_7), J10.8 (Pin_8), J10.9 (Pin_9)
- net MISO: now also U1.21 (GPIO16)
- net MOSI: now also U1.25 (GPIO19)
- net SCL_Bus_0: now also U1.27 (GPIO21); no longer U1.22 (GPIO17)
- net SDA_Bus_0: now also U1.26 (GPIO20); no longer U1.21 (GPIO16)
- net Switch_Interrupt: now also U1.20 (GPIO15), J8.1 (Pin_1); no longer U5.13 (~{INT})
- new net: J7.1 (Pin_1), U5.13 (~{INT})
- no-connect marks 9 -> 70

Commit message: TO-DO: fix silkscreen
Parts:
- added JP15: SolderJumper_2_Open, Jumper:SolderJumper-2_P1.3mm_Open_RoundedPad1.0x1.5mm, symbol Jumper:SolderJumper_2_Open
Connections:
- net +3V3: now also JP15.1 (A); no longer J9.10 (Pin_10), J9.11 (Pin_11), J9.12 (Pin_12), J9.13 (Pin_13), J9.14 (Pin_14), J9.8 (Pin_8), J9.9 (Pin_9)
- new net: J9.10 (Pin_10), J9.11 (Pin_11), J9.12 (Pin_12), J9.13 (Pin_13), J9.14 (Pin_14), J9.8 (Pin_8), J9.9 (Pin_9), JP15.2 (B)
Changed lines of the file:
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@@
 	)
 	(junction
-		(at 425.45 168.91)
-		(diameter 0)
-		(color 0 0 0 0)
-	)
-	(junction
 		(at 444.5 184.15)
 		(diameter 0)
@@
 	)
 	(junction
-		(at 425.45 166.37)
-		(diameter 0)
-		(color 0 0 0 0)
-	)
-	(junction
 		(at 49.53 168.91)
 		(diameter 0)
@@
 	)
 	(junction
-		(at 425.45 151.13)
-		(diameter 0)
-		(color 0 0 0 0)
-	)
-	(junction
 		(at 425.45 161.29)
 		(diameter 0)
@@
 	)
 	(junction
+		(at 425.45 184.15)
+		(diameter 0)
+		(color 0 0 0 0)
+	)
+	(junction
 		(at 154.94 266.7)
 		(diameter 0)
@@
 	(wire
 		(pts
+			(xy 425.45 163.83) (xy 425.45 166.37)
+		)
+		(stroke
+			(width 0)
+			(type default)
+		)
+	)
+	(wire
+		(pts
 			(xy 458.47 26.67) (xy 458.47 43.18)
 		)
@@
 	(wire
 		(pts
+			(xy 425.45 171.45) (xy 427.99 171.45)
+		)
+		(stroke
+			(width 0)
+			(type default)
+		)
+	)
+	(wire
+		(pts
 			(xy 121.92 287.02) (xy 116.84 287.02)
 		)
@@
 	(wire
 		(pts
+			(xy 427.99 163.83) (xy 425.45 163.83)
+		)
+		(stroke
+			(width 0)
+			(type default)
+		)
+	)
+	(wire
+		(pts
 			(xy 49.53 147.32) (xy 80.01 147.32)
 		)
@@
 	(wire
 		(pts
-			(xy 425.45 166.37) (xy 425.45 168.91)
-		)
-		(stroke
-			(width 0)
-			(type default)
-		)
-	)
-	(wire
-		(pts
 			(xy 179.07 151.13) (xy 179.07 149.86)
 		)
@@
 	(wire
 		(pts
+			(xy 425.45 193.04) (xy 425.45 184.15)
+		)
+		(stroke
+			(width 0)
+			(type default)
+		)
+	)
+	(wire
+		(pts
 			(xy 58.42 54.61) (xy 35.56 54.61)
 		)
@@
 	(wire
 		(pts
-			(xy 425.45 163.83) (xy 425.45 166.37)
-		)
-		(stroke
-			(width 0)
-			(type default)
-		)
-	)
-	(wire
-		(pts
 			(xy 233.68 74.93) (xy 240.03 74.93)
 		)
@@
 	(wire
 		(pts
-			(xy 425.45 146.05) (xy 425.45 151.13)
-		)
-		(stroke
-			(width 0)
-			(type default)
-		)
-	)
-	(wire
-		(pts
 			(xy 322.58 83.82) (xy 322.58 85.09)
 		)
@@
 	)
 	(label "+3V3"
-		(at 425.45 146.05 0)
+		(at 425.45 193.04 0)
 		(fields_autoplaced yes)
 		(effects
@@
 					(unit 1)
 				)
+			)
+		)
+	)
+	(symbol
+		(lib_id "Jumper:SolderJumper_2_Open")
+		(at 427.99 167.64 90)
+		(unit 1)
+		(exclude_from_sim yes)
+		(in_bom no)
+		(on_board yes)
+		(dnp no)
+		(fields_autoplaced yes)
+		(property "Reference" "JP15"
+			(at 430.53 166.3699 90)
+			(effects
+				(font
+					(size 1.27 1.27)
+				)
+				(justify right)
+			)
+		)
+		(property "Value" "SolderJumper_2_Open"
+			(at 430.53 168.9099 90)
+			(effects
+				(font
+					(size 1.27 1.27)
+				)
+				(justify right)
+			)
+		)
+		(property "Footprint" "Jumper:SolderJumper-2_P1.3mm_Open_RoundedPad1.0x1.5mm"
+			(at 427.99 167.64 0)
+			(effects
+				(font
+					(size 1.27 1.27)
+				)
+				(hide yes)
+			)
+		)
+		(property "Datasheet" "~"
+			(at 427.99 167.64 0)
+			(effects
+				(font
+					(size 1.27 1.27)
+				)
+				(hide yes)
+			)
+		)
+		(property "Description" "Solder Jumper, 2-pole, open"
+			(at 427.99 167.64 0)
+			(effects
+				(font
+					(size 1.27 1.27)
+				)
+				(hide yes)
+			)
+		)
+		(pin "2"
+		)
+		(pin "1"
+		)
+		(instances
+			(project ""
+				(path "/ae16032a-0ba6-4513-ba96-439785199ac8"
+					(reference "JP15")
+					(unit 1)
+				)

Commit message: Finished layout, no errors in DRC, silkscreen aso finished
Connections:
- net +3V3: now also JP11.3 (B); no longer JP11.1 (A)
- net GND: now also JP11.1 (A); no longer J1.1 (Pin_1), JP11.3 (B)
- net SCL_Bus_1: now also J11.1 (Pin_1)
- net SDA_Bus_1: now also J12.1 (Pin_1)
- no-connect marks 70 -> 69
Other:
- note added: "SCK does not need to be connected; The sck jumper in the module must be connected to gnd"
Changed lines of the file:
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@@
 	)
 	(no_connect
-		(at 482.6 184.15)
-	)
-	(no_connect
 		(at 283.21 190.5)
 	)
@@
 	)
 	(no_connect
+		(at 179.07 31.75)
+	)
+	(no_connect
 		(at 463.55 153.67)
 	)
@@
 	)
 	(no_connect
-		(at 463.55 184.15)
-	)
-	(no_connect
 		(at 501.65 166.37)
 	)
@@
 	(wire
 		(pts
-			(xy 179.07 31.75) (xy 185.42 31.75)
-		)
-		(stroke
-			(width 0)
-			(type default)
-		)
-	)
-	(wire
-		(pts
 			(xy 52.07 62.23) (xy 58.42 62.23)
 		)
@@
 		)
 	)
+	(text "SCK does not need \nto be connected;\nThe sck jumper in \nthe module must be \nconnected to gnd\n"
+		(exclude_from_sim no)
+		(at 163.83 33.02 0)
+		(effects
+			(font
+				(size 0.6 0.6)
+			)
+			(justify left)
+		)
+	)
 	(text "The output capacitor should have an \neffective series resistance greater \nthan 0.1Ω and less than 5Ω, and a \nresonant frequency above 1 MHz."
 		(exclude_from_sim no)
@@
 		)
 	)
+	(label "SCL_Bus_1"
+		(at 463.55 184.15 0)
+		(fields_autoplaced yes)
+		(effects
+			(font
+				(size 1.27 1.27)
+			)
+			(justify left bottom)
+		)
+	)
 	(label "Encoder1_A"
 		(at 314.96 261.62 0)
@@
 		)
 	)
+	(label "SDA_Bus_1"
+		(at 482.6 184.15 0)
+		(fields_autoplaced yes)
+		(effects
+			(font
+				(size 1.27 1.27)
+			)
+			(justify left bottom)
+		)
+	)
 	(label "Pin1"
 		(at 123.19 285.75 0)
@@
 		)
 	)
-	(label "SCK"
-		(at 185.42 31.75 180)
-		(fields_autoplaced yes)
-		(effects
-			(font
-				(size 1.27 1.27)
-			)
-			(justify right bottom)
-		)
-	)
 	(label "CLK"
 		(at 240.03 74.93 180)
@@
 		(lib_id "Jumper:SolderJumper_3_Bridged12")
 		(at 54.61 168.91 0)
+		(mirror y)
 		(unit 1)
 		(exclude_from_sim no)
@@
 					(unit 1)
 				)
+			)
+		)
+	)
+	(symbol
+		(lib_id "Graphic:Logo_Open_Hardware_Large")
+		(at 186.69 110.49 0)
+		(unit 1)
+		(exclude_from_sim no)
+		(in_bom yes)
+		(on_board yes)
+		(dnp no)
+		(fields_autoplaced yes)
+		(property "Reference" "#SYM1"
+			(at 186.69 97.79 0)
+			(effects
+				(font
+					(size 1.27 1.27)
+				)
+				(hide yes)
+			)
+		)
+		(property "Value" "Logo_Open_Hardware_Large"
+			(at 186.69 120.65 0)
+			(effects
+				(font
+					(size 1.27 1.27)
+				)
+				(hide yes)
+			)
+		)
+		(property "Footprint" "Symbol:OSHW-Logo2_14.6x12mm_SilkScreen"
+			(at 186.69 110.49 0)
+			(effects
+				(font
+					(size 1.27 1.27)
+				)
+				(hide yes)
+			)
+		)
+		(property "Datasheet" "~"
+			(at 186.69 110.49 0)
+			(effects
+				(font
+					(size 1.27 1.27)
+				)
+				(hide yes)
+			)
+		)
+		(property "Description" "Open Hardware logo, large"
+			(at 186.69 110.49 0)
+			(effects
+				(font
+					(size 1.27 1.27)
+				)
+				(hide yes)
+			)
+		)
+		(property "Sim.Enable" "0"
+			(at 186.69 110.49 0)
+			(effects
+				(font
+					(size 1.27 1.27)
+				)
+				(hide yes)
+			)
+		)
+		(instances
+			(project ""
+				(path "/ae16032a-0ba6-4513-ba96-439785199ac8"
+					(reference "#SYM1")
+					(unit 1)
+				)
