File: hardware/electronics/PicoSynth.kicad_pcb (KiCad board)
At the start: 2 copper layers, 164 x 82.4 mm, 151 parts, among them J1 Conn_01x06_Socket, J10 Conn_01x14_Socket, J11 Conn_01x14_Socket, J12 Conn_01x14_Socket, J13 Conn_01x14_Socket, J14 Conn_01x14_Socket, J3 Conn_01x04_Socket, J4 Conn_01x09_Socket, J5 Line_Out, J6 Conn_01x06_Socket, J7 Conn_01x01_Socket, J8 Conn_01x01_Socket, J9 Conn_01x14_Socket, SW1 RotaryEncoder_Switch_MP, SW10 SW_Push_45deg, SW11 SW_Push_45deg, SW12 SW_Push_45deg, SW13 SW_Push_45deg, SW14 SW_Push_45deg, SW15 SW_Push_45deg, SW16 SW_Push_45deg, SW17 SW_Push_45deg, SW18 SW_Push_45deg, SW19 SW_Push_45deg, SW2 RotaryEncoder_Switch_MP, SW20 SW_Push_45deg, SW3 RotaryEncoder_Switch_MP, SW4 RotaryEncoder_Switch_MP, SW5 SW_Push_45deg, SW6 SW_Push_45deg, SW7 SW_Push_45deg, SW8 SW_Push_45deg, SW9 SW_Push_45deg, U1 Pico, U5 PCF8574, U6 PCF8574, U7 PCF8574, U8 AMS1117-3.3

Commit message: Ready to order
Other:
- board text added: "A0"
- board text added: "A1"
- board text added: "A2"
- board text added: "Matrix Interrupt"
Changed lines of the file:
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@@
 			(plotinvisibletext no)
 			(sketchpadsonfab no)
-			(subtractmaskfromsilk no)
+			(subtractmaskfromsilk yes)
 			(outputformat 1)
 			(mirror no)
-			(drillshape 1)
+			(drillshape 0)
 			(scaleselection 1)
-			(outputdirectory "")
+			(outputdirectory "Fab/")
 		)
 	)
@@
 		(layer "Edge.Cuts")
 	)
+	(gr_text "Matrix \nInterrupt"
+		(at 92.202 36.7284 0)
+		(layer "B.SilkS")
+		(effects
+			(font
+				(size 1 1)
+				(thickness 0.153)
+			)
+			(justify left bottom mirror)
+		)
+	)
+	(gr_text "A2\n"
+		(at 143.7386 57.7088 0)
+		(layer "B.SilkS")
+		(effects
+			(font
+				(size 1 1)
+				(thickness 0.153)
+			)
+			(justify left bottom mirror)
+		)
+	)
+	(gr_text "A0"
+		(at 115.2398 55.8292 0)
+		(layer "B.SilkS")
+		(effects
+			(font
+				(size 1 1)
+				(thickness 0.153)
+			)
+			(justify left bottom mirror)
+		)
+	)
+	(gr_text "A1\n"
+		(at 157.099 55.7022 0)
+		(layer "B.SilkS")
+		(effects
+			(font
+				(size 1 1)
+				(thickness 0.153)
+			)
+			(justify left bottom mirror)
+		)
+	)
 	(gr_text "GND"
 		(at 169.418 67.183 0)
@@
 		)
 	)
+	(gr_text "A0"
+		(at 151.9428 55.7276 0)
+		(layer "B.SilkS")
+		(effects
+			(font
+				(size 1 1)
+				(thickness 0.153)
+			)
+			(justify left bottom mirror)
+		)
+	)
+	(gr_text "A2\n"
+		(at 162.7378 55.6514 0)
+		(layer "B.SilkS")
+		(effects
+			(font
+				(size 1 1)
+				(thickness 0.153)
+			)
+			(justify left bottom mirror)
+		)
+	)
+	(gr_text "A2\n"
+		(at 125.5014 55.7276 0)
+		(layer "B.SilkS")
+		(effects
+			(font
+				(size 1 1)
+				(thickness 0.153)
+			)
+			(justify left bottom mirror)
+		)
+	)
 	(gr_text "+3V3\n"
 		(at 169.672 54.483 0)
@@
 		)
 	)
+	(gr_text "A1\n"
+		(at 138.4554 57.7596 0)
+		(layer "B.SilkS")
+		(effects
+			(font
+				(size 1 1)
+				(thickness 0.153)
+			)
+			(justify left bottom mirror)
+		)
+	)
+	(gr_text "A0"
+		(at 133.4262 57.8358 0)
+		(layer "B.SilkS")
+		(effects
+			(font
+				(size 1 1)
+				(thickness 0.153)
+			)
+			(justify left bottom mirror)
+		)
+	)
 	(gr_text "SDA"
 		(at 169.545 62.103 0)
@@
 			)
 			(justify left bottom mirror)
+		)
+	)
+	(gr_text "A1\n"
+		(at 120.4214 55.753 0)
+		(layer "B.SilkS")
+		(effects
+			(font
+				(size 1 1)
+				(thickness 0.153)
+			)
+			(justify left bottom mirror)
